File: e7_BMS_PDU/12V_OUT.kicad_sch (KiCad schematic)
At the start: 29 parts, among them SW1 EN, U3 LM70660RRXR, U5 SKA60A-12

Commit message: updated files
Connections:
- net at U3.11 (ISNS+): now also L1.2, R49.1
Other:
- moved on the sheet: R49
Changed lines of the file:
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@@
 	)
 	(junction
+		(at 204.47 44.45)
+		(diameter 0)
+		(color 0 0 0 0)
+	)
+	(junction
 		(at 151.13 92.71)
 		(diameter 0)
@@
 	(wire
 		(pts
-			(xy 199.39 44.45) (xy 199.39 54.61)
+			(xy 204.47 44.45) (xy 204.47 54.61)
 		)
 		(stroke
@@
 	(wire
 		(pts
-			(xy 210.82 44.45) (xy 215.9 44.45)
+			(xy 212.09 44.45) (xy 215.9 44.45)
 		)
 		(stroke
@@
 	(wire
 		(pts
+			(xy 204.47 44.45) (xy 203.2 44.45)
+		)
+		(stroke
+			(width 0)
+			(type default)
+		)
+	)
+	(wire
+		(pts
 			(xy 106.68 152.4) (xy 106.68 149.86)
 		)
@@
 	(wire
 		(pts
-			(xy 151.13 54.61) (xy 199.39 54.61)
+			(xy 151.13 54.61) (xy 204.47 54.61)
 		)
 		(stroke
@@
 	(symbol
 		(lib_id "Device:R")
-		(at 207.01 44.45 90)
+		(at 208.28 44.45 90)
 		(unit 1)
 		(exclude_from_sim no)
@@
 		(fields_autoplaced yes)
 		(property "Reference" "R49"
-			(at 207.01 38.1 90)
+			(at 208.28 38.1 90)
 			(effects
 				(font
@@
 		)
 		(property "Value" "6m"
-			(at 207.01 40.64 90)
+			(at 208.28 40.64 90)
 			(effects
 				(font
@@
 		)
 		(property "Footprint" "Resistor_SMD:R_2512_6332Metric"
-			(at 207.01 46.228 90)
+			(at 208.28 46.228 90)
 			(effects
 				(font
@@
 		)
 		(property "Datasheet" "~"
-			(at 207.01 44.45 0)
+			(at 208.28 44.45 0)
 			(effects
 				(font
@@
 		)
 		(property "Description" "Resistor"
-			(at 207.01 44.45 0)
+			(at 208.28 44.45 0)
 			(effects
 				(font
