File: e7_BMS_PDU/e7_BMS_PDU.kicad_sch (KiCad schematic)
At the start: 45 parts, among them J13 Conn_01x05, J14 XT60PW-M, J15 XT60PW-M, J16 CAN, J2 CAN, Q1 MMBTA05, U4 STM32G0B1KETx, U6 TLV76733DRVx, U7 ISO1044BD, U8 USBLC6-2SC6

Commit message: updated files
Parts:
- added C36: 220uF, Capacitor_SMD:CP_Elec_8x10.5, symbol Device:C_Polarized
- added D2, D3, D4: Red, PCM_JLCPCB:D_0603, symbol PCM_JLCPCB-Diodes:LED,0603,Red
- added D6: SMCJ7.0CA, PCM_JLCPCB:D_SMC, symbol PCM_JLCPCB-Diodes:TVS-Bi,SMCJ7.0CA
- added F2: 5A 2920, Fuse:Fuse_2920_7451Metric, symbol Device:Fuse
- added J3: XT60PW-M, Connector_AMASS:AMASS_XT60PW-M_1x02_P7.20mm_Horizontal, symbol Connector_Generic:Conn_01x02
- added L3: 470nH,3.7A, PCM_JLCPCB:L_1008, symbol PCM_JLCPCB-Inductors:470nH,3.7A
- added R55, R56: 4.7kΩ, PCM_JLCPCB:R_0603, symbol PCM_JLCPCB-Resistors:0603,4.7kΩ
- added R57: 1kΩ, PCM_JLCPCB:R_0603, symbol PCM_JLCPCB-Resistors:0603,1kΩ
- added U9: SKE15, SKE15:VREG_SKE15, symbol SKE15:SKE15
Connections:
- net +12V: now also J3.2 (Pin_2), R55.1, U9.1 (+VIN)
- net +3.3V: now also R57.2
- net +5V: now also D6.2, F2.2, R56.1
- net GND2: now also D2.1, D4.1, J3.1 (Pin_1), U9.2 (-VIN)
- net GND3: now also C36.2, D3.1, D6.1, U9.5 (-VOUT)
- net VBAT: now also U2.3 (VC16), U2.5 (VC15), U2.7 (VC14), U2.9 (VC13)
- new net: C36.1, F2.1, L3.2
- new net: D3.2, R56.2
- new net: D4.2, R57.1
- new net: D2.2, R55.2
- new net: L3.1, U9.3 (+VOUT)
- no-connect marks 43 -> 39
Other:
- note added: "power indication LEDs"
